Commit message: Completed RViz Setup. Need to incorporate controllers

File: friday_description/urdf/friday.urdf.xacro (robot description, xacro)
@@ -18,8 +18,8 @@
 	<!-- Properties -->
     <xacro:property name="PI" value="3.14159265359" />
-    <xacro:property name="arm_offset_y" value="0" />
-    <xacro:property name="arm_offset_z" value="7" />
-    <xacro:property name="main_origin_height" value="202.628" />
-    <xacro:property name="second_origin_height" value="260.5" />
+    <xacro:property name="arm_offset_y" value="-0.022" />
+    <xacro:property name="arm_offset_z" value="-0.023" />
+    <xacro:property name="main_origin_height" value="0.202628" />
+    <xacro:property name="second_origin_height" value="0.26050" />
     <xacro:property name="base_lower_limit" value="${-PI}" />
     <xacro:property name="base_upper_limit" value="${PI}" />
@@ -40,5 +40,5 @@
 			<origin xyz="0 0 0" rpy="0 0 0" />
             <geometry>
-                <mesh filename="package://friday_description/meshes/stl/base_fix.stl" />
+                <mesh filename="package://friday_description/meshes/dae/base_fix.dae" />
             </geometry>
         </collision>
